File: _autosave-solar_light.kicad_pcb (KiCad board)
At the start: 2 copper layers, 26 parts, among them J1 Solar Cell, J2 Battery, J3 breakout header, J4 USB_B_Mini, SW1 SW_SPST, SW2 BRIGHTNESS, SW3 COLOR, U1 ATSAMD21E18A-MU, U2 MC34673, U3 ISL9111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

Commit message: schematic done; pcb started
Parts:
- D1, D2: moved to B.Cu
- J1: value Solar Cell -> SOL
- J2: value Battery -> BATT
- J3: footprint Connector_PinHeader_1.00mm:PinHeader_1x08_P1.00mm_Horizontal -> Connector_PinHeader_1.00mm:PinHeader_1x08_P1.00mm_Vertical
- J4: footprint Connector_USB:USB_Micro-B_Amphenol_10103594-0001LF_Horizontal -> Connector_USB:USB_Micro-B_Amphenol_10103594-0001LF_Horizontal-no-th
- SW1: value SW_SPST -> RESET; footprint Button_Switch_THT:SW_PUSH_6mm -> Button_Switch_THT:SW_PUSH_3.5mm
- SW2: value BRIGHTNESS -> BRT; footprint Button_Switch_THT:SW_PUSH_6mm -> Button_Switch_THT:SW_PUSH_3.5mm
- SW3: value COLOR -> COL; footprint Button_Switch_THT:SW_PUSH_6mm -> Button_Switch_THT:SW_PUSH_3.5mm
- moved SW3 69.6 mm to (156.8, 129.0), turned to 90 degrees
- moved C1 68.2 mm to (180.1, 123.8)
- moved L1 68.2 mm to (171.2, 124.7)
- moved U1 60.3 mm to (139.9, 127.9)
- moved SW2 55.4 mm to (157.2, 112.2), turned to 270 degrees
- moved J4 55.1 mm to (155.8, 120.6), turned to 90 degrees
- moved J3 51.8 mm to (134.8, 124.4)
- moved U3 48.6 mm to (144.6, 121.0)
- moved SW1 47.8 mm to (137.3, 109.6), turned to 180 degrees
- moved TP2 47.3 mm to (140.0, 121.8)
- moved C3 47.0 mm to (166.0, 119.5)
- moved C6 47.0 mm to (174.6, 111.6)
- moved C2 47.0 mm to (174.6, 110.1)
- moved C4 47.0 mm to (168.4, 117.5)
- moved C5 47.0 mm to (166.0, 121.0)
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Routing:
- net GND: track 0.00 -> 5.52 mm
- net Net-(J3-Pad8): track 0.00 -> 3.37 mm
- net Net-(J3-Pad1): track 0.00 -> 3.34 mm
- net Net-(J3-Pad7): track 0.00 -> 3.16 mm
- net Net-(J3-Pad2): track 0.00 -> 3.13 mm
- net Net-(J3-Pad6): track 0.00 -> 2.96 mm
- net Net-(J3-Pad3): track 0.00 -> 2.92 mm
- net Net-(J3-Pad5): track 0.00 -> 2.75 mm
- net Net-(J3-Pad4): track 0.00 -> 2.72 mm
- added copper zone on F.Cu, net GND
Other:
- board outline added: 25 x 25 mm
