File: _saved_solar_light.sch (KiCad schematic (older format))
At the start: 26 parts, among them J1 Solar Cell, J2 Battery, SW1 SW_SPST, SW2 BRIGHTNESS, SW3 COLOR, U1 ATSAMD21E18A-MU, U2 MC34673, U3 ISL9113, U4 MIC3490-3v3

Commit message: schematic done; pcb started
Parts:
- removed U3: ISL9113, symbol solar_light:ISL9113
- added U3: ISL9111, Package_TO_SOT_SMD:SOT-23-6, symbol solar_light:ISL9111
- C1, C2, C3, C4, C5, C6: footprint (none) -> Capacitor_SMD:C_0603_1608Metric
- D3: footprint (none) -> Diode_SMD:D_SOD-123
- J1, J2: footprint (none) -> Connector_PinHeader_1.00mm:PinHeader_1x02_P1.00mm_Vertical
- J3: renamed from J?; value Conn_01x08_Female -> breakout header; footprint (none) -> Connector_PinHeader_1.00mm:PinHeader_1x08_P1.00mm_Horizontal
- J4: renamed from J?; footprint (none) -> Connector_USB:USB_Micro-B_Amphenol_10103594-0001LF_Horizontal-no-th
- L1: value 2.2uh -> 4.7uH; footprint (none) -> Resistor_SMD:R_0603_1608Metric_Pad1.05x0.95mm_HandSolder
- R1: footprint (none) -> Resistor_SMD:R_0603_1608Metric
- R2, R3: renamed from R?; footprint (none) -> Resistor_SMD:R_0603_1608Metric
- SW1, SW2, SW3: footprint (none) -> Button_Switch_THT:SW_PUSH_3.5mm
- TP1, TP2: footprint (none) -> TestPoint:TestPoint_Pad_D1.5mm
- U1: footprint QFN50P500X500X100-33N -> Package_DFN_QFN:QFN-32-1EP_5x5mm_P0.5mm_EP3.6x3.6mm
- U4: footprint (none) -> Package_TO_SOT_SMD:SOT-23-5
Connections:
- net 5v: now also C2.1, U3.5 (Vout); no longer C6.1
- net GND: now also U3.2 (GND)
- net VCC: now also C6.1, L1.2, U3.3 (EN), U3.6 (Vin); no longer C2.1, L1.1
- new net: L1.1, U3.1 (SW)
Other:
- moved on the sheet: L1
