File: solar_light.kicad_pcb (KiCad board)
At the start: 2 copper layers, 26 parts, among them J1 Solar Cell, J2 Battery, J3 breakout header, J4 USB_B_Mini, SW1 SW_SPST, SW2 BRIGHTNESS, SW3 COLOR, U1 ATSAMD21E18A-MU, U2 MC34673, U3 ISL9111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

Commit message: routed!
Parts:
- removed R3: R_Small, Resistor_SMD:R_0603_1608Metric
- added ?: R_Small, Resistor_SMD:R_0603_1608Metric, F.Cu at (150.8, 121.4)
- D1, D2: moved to B.Cu
- J1: value Solar Cell -> SOL
- J2: value Battery -> BATT
- J3: footprint Connector_PinHeader_1.00mm:PinHeader_1x08_P1.00mm_Horizontal -> Connector_PinHeader_1.00mm:PinHeader_1x08_P1.00mm_Vertical
- J4: footprint Connector_USB:USB_Micro-B_Amphenol_10103594-0001LF_Horizontal -> Connector_USB:USB_Micro-B_Amphenol_10103594-0001LF_Horizontal-no-th
- SW1: value SW_SPST -> RESET; footprint Button_Switch_THT:SW_PUSH_6mm -> Button_Switch_THT:SW_PUSH_3.5mm
- SW2: value BRIGHTNESS -> BRT; footprint Button_Switch_THT:SW_PUSH_6mm -> Button_Switch_THT:SW_PUSH_3.5mm
- SW3: value COLOR -> COL; footprint Button_Switch_THT:SW_PUSH_6mm -> Button_Switch_THT:SW_PUSH_3.5mm
- U4: value MIC3490-3v3 -> MIC3490
- moved SW3 69.6 mm to (156.8, 129.0), turned to 90 degrees
- moved U1 60.3 mm to (139.9, 127.9)
- moved C2 57.6 mm to (151.4, 129.2)
- moved U3 56.9 mm to (147.2, 128.9)
- moved SW2 55.4 mm to (157.2, 112.2), turned to 270 degrees
- moved J4 55.1 mm to (155.8, 120.6), turned to 90 degrees
- moved C6 54.5 mm to (151.4, 127.6)
- moved L1 52.4 mm to (147.3, 125.9)
- moved J3 51.8 mm to (134.8, 124.4)
- moved U4 48.9 mm to (144.4, 122.5), turned to 180 degrees
- moved C4 47.8 mm to (151.4, 125.9)
- moved SW1 47.8 mm to (137.3, 109.6), turned to 180 degrees
- moved TP2 46.0 mm to (135.1, 119.2)
- moved D3 43.6 mm to (139.8, 118.8), turned to 180 degrees
- moved D2 43.5 mm to (146.1, 121.9)
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Routing:
- net VCC: track 0.00 -> 43.9 mm
- net /5v: track 0.00 -> 28.6 mm, vias 0 -> 1
- net Net-(SW2-Pad2): track 0.00 -> 25.8 mm, vias 0 -> 1
- net /light: track 0.00 -> 22.9 mm, vias 0 -> 1
- net Net-(SW2-Pad1): track 0.00 -> 22.0 mm, vias 0 -> 1
- net Net-(SW3-Pad1): track 0.00 -> 16.9 mm
- net Net-(SW1-Pad2): track 0.00 -> 16.7 mm, vias 0 -> 1
- net /3v3: track 0.00 -> 15.8 mm, vias 0 -> 2
- net Net-(SW3-Pad2): track 0.00 -> 15.5 mm
- net GND: track 0.00 -> 15.1 mm, vias 0 -> 2
- net /D+: track 0.00 -> 10.6 mm
- net /D-: track 0.00 -> 9.81 mm
- net Net-(D1-Pad2): track 0.00 -> 9.46 mm, vias 0 -> 2
- net Net-(TP2-Pad1): track 0.00 -> 7.71 mm
- net /Solar+: track 0.00 -> 6.38 mm
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- added copper zone on F.Cu, net GND
Other:
- board outline added: 25 x 25 mm
- net class Default: clearance 0.2 -> 0.15; trace_width 0.25 -> 0.15; via_drill 0.4 -> 0.254
- rule trace_clearance: 0.2 -> 0.15
- rule trace_min: 0.2 -> 0.15
- rule via_min_drill: 0.3 -> 0.254
- rule via_min_size: 0.4 -> 0.381
