File: solar_light.sch (KiCad schematic (older format))
At the start: 4 parts, among them U1 ATTINY-1616MNR, U2 MC34673

Commit message: wip
Parts:
- added C?: C_Small, symbol Device:C_Small
- added D?: D_Schottky_Small, symbol Device:D_Schottky_Small
- added J?: Battery, symbol Connector:Conn_01x02_Female
- added J?: Solar Cell, symbol Connector:Conn_01x02_Female
- added R?: R_Small, symbol Device:R_Small
- D? (x2): symbol LED:WS2812B -> solar_light-rescue:WS2812B-LED
- U1: symbol solar_light:ATTINY-1616MNR -> solar_light-rescue:ATTINY-1616MNR-solar_light
- U2: symbol Battery_Management:MC34673 -> solar_light-rescue:MC34673-Battery_Management
Connections:
- net labels added: GND, Solar+, VCC
- wire segments 3 -> 18
Changed lines of the file:
@@
 EESchema Schematic File Version 4
-EELAYER 26 0
+LIBS:solar_light-cache
+EELAYER 29 0
 EELAYER END
 $Descr A4 11693 8268
@@
 $EndDescr
 $Comp
-L solar_light:ATTINY-1616MNR U1
+L solar_light-rescue:ATTINY-1616MNR-solar_light U1
 U 1 1 5C9202C7
 P 1350 2450
@@
 $EndComp
 $Comp
-L Battery_Management:MC34673 U2
+L solar_light-rescue:MC34673-Battery_Management U2
 U 1 1 5C9207F0
 P 7500 1800
@@
 $EndComp
 $Comp
-L LED:WS2812B D?
+L solar_light-rescue:WS2812B-LED D?
 U 1 1 5C920A2F
 P 4150 5400
@@
 $EndComp
 $Comp
-L LED:WS2812B D?
+L solar_light-rescue:WS2812B-LED D?
 U 1 1 5C920B0C
 P 5150 5400
@@
 Wire Wire Line
 	4450 5400 4850 5400
+$Comp
+L Connector:Conn_01x02_Female J?
+U 1 1 5CAC0189
+P 9500 1400
+F 0 "J?" H 9528 1376 50  0000 L CNN
+F 1 "Battery" H 9528 1285 50  0000 L CNN
+F 2 "" H 9500 1400 50  0001 C CNN
+F 3 "~" H 9500 1400 50  0001 C CNN
+	1    9500 1400
+	1    0    0    -1
+$EndComp
+$Comp
+L Connector:Conn_01x02_Female J?
+U 1 1 5CAC0F37
+P 6900 1100
+F 0 "J?" H 6928 1076 50  0000 L CNN
+F 1 "Solar Cell" H 6928 985 50  0000 L CNN
+F 2 "" H 6900 1100 50  0001 C CNN
+F 3 "~" H 6900 1100 50  0001 C CNN
+	1    6900 1100
+	-1   0    0    1
+$EndComp
+$Comp
+L Device:D_Schottky_Small D?
+U 1 1 5CAC133A
+P 8900 1400
+F 0 "D?" H 8900 1605 50  0000 C CNN
+F 1 "D_Schottky_Small" H 8900 1514 50  0000 C CNN
+F 2 "" V 8900 1400 50  0001 C CNN
+F 3 "~" V 8900 1400 50  0001 C CNN
+	1    8900 1400
+	1    0    0    -1
+$EndComp
+Wire Wire Line
+	9000 1400 9050 1400
+Wire Wire Line
+	8000 1400 8000 1500
+$Comp
+L power:GND #PWR?
+U 1 1 5CAC36C8
+P 9300 1650
+F 0 "#PWR?" H 9300 1400 50  0001 C CNN
+F 1 "GND" H 9305 1477 50  0000 C CNN
+F 2 "" H 9300 1650 50  0001 C CNN
+F 3 "" H 9300 1650 50  0001 C CNN
+	1    9300 1650
+	1    0    0    -1
+$EndComp
+Wire Wire Line
+	9300 1500 9300 1600
+$Comp
+L power:GND #PWR?
+U 1 1 5CAC3D1E
+P 7850 1000
+F 0 "#PWR?" H 7850 750 50  0001 C CNN
+F 1 "GND" H 7855 827 50  0000 C CNN
+F 2 "" H 7850 1000 50  0001 C CNN
+F 3 "" H 7850 1000 50  0001 C CNN
+	1    7850 1000
+	1    0    0    -1
+$EndComp
+$Comp
+L power:GND #PWR?
+U 1 1 5CAC4E25
+P 7500 2450
+F 0 "#PWR?" H 7500 2200 50  0001 C CNN
+F 1 "GND" H 7505 2277 50  0000 C CNN
+F 2 "" H 7500 2450 50  0001 C CNN
+F 3 "" H 7500 2450 50  0001 C CNN
+	1    7500 2450
+	1    0    0    -1
+$EndComp
+Wire Wire Line
+	7400 2300 7500 2300
+Connection ~ 7500 2300
+$Comp
+L Device:C_Small C?
+U 1 1 5CAC5C29
+P 9050 1500
+F 0 "C?" H 9142 1546 50  0000 L CNN
+F 1 "C_Small" H 9142 1455 50  0000 L CNN
+F 2 "" H 9050 1500 50  0001 C CNN
+F 3 "~" H 9050 1500 50  0001 C CNN
+	1    9050 1500
+	1    0    0    -1
+$EndComp
+Connection ~ 9050 1400
+Wire Wire Line
+	9050 1400 9300 1400
+Wire Wire Line
+	9050 1600 9300 1600
+Wire Wire Line
+	7500 2300 7500 2450
+Connection ~ 9300 1600
+Wire Wire Line
+	9300 1600 9300 1650
+Wire Wire Line
+	8000 1700 8000 1800
+Text Label 8100 1700 0    50   ~ 0
+Solar+
+Wire Wire Line
+	8100 1700 8000 1700
+Connection ~ 8000 1700
+Text Label 7000 1800 2    50   ~ 0
+Solar+
+Text Label 7500 1300 0    50   ~ 0
+Solar+
+Text Label 7100 1100 0    50   ~ 0
+Solar+
+Wire Wire Line
+	7850 1000 7100 1000
+$Comp
+L power:GND #PWR?
+U 1 1 5CACB124
+P 8300 2250
+F 0 "#PWR?" H 8300 2000 50  0001 C CNN
+F 1 "GND" H 8305 2077 50  0000 C CNN
+F 2 "" H 8300 2250 50  0001 C CNN
+F 3 "" H 8300 2250 50  0001 C CNN
+	1    8300 2250
+	1    0    0    -1
+$EndComp
+$Comp
+L Device:R_Small R?
+U 1 1 5CACB93D
+P 8200 2100
+F 0 "R?" V 8004 2100 50  0000 C CNN
+F 1 "R_Small" V 8095 2100 50  0000 C CNN
+F 2 "" H 8200 2100 50  0001 C CNN
+F 3 "~" H 8200 2100 50  0001 C CNN
+	1    8200 2100
+	0    1    1    0
+$EndComp
+Wire Wire Line
+	8000 2100 8100 2100
+Wire Wire Line
+	8300 2100 8300 2250
+$Comp
+L power:VCC #PWR?
+U 1 1 5CACCD8D
+P 8000 1400
+F 0 "#PWR?" H 8000 1250 50  0001 C CNN
+F 1 "VCC" H 8017 1573 50  0000 C CNN
+F 2 "" H 8000 1400 50  0001 C CNN
+F 3 "" H 8000 1400 50  0001 C CNN
+	1    8000 1400
+	1    0    0    -1
+$EndComp
+$Comp
+L power:VCC #PWR?
+U 1 1 5CACD3A2
+P 8800 1400
+F 0 "#PWR?" H 8800 1250 50  0001 C CNN
+F 1 "VCC" H 8818 1573 50  0000 C CNN
+F 2 "" H 8800 1400 50  0001 C CNN
+F 3 "" H 8800 1400 50  0001 C CNN
+	1    8800 1400
+	-1   0    0    1
+$EndComp
+$Comp
+L power:VCC #PWR?
+U 1 1 5CACDC33
+P 2100 1550
+F 0 "#PWR?" H 2100 1400 50  0001 C CNN
+F 1 "VCC" H 2117 1723 50  0000 C CNN
+F 2 "" H 2100 1550 50  0001 C CNN
+F 3 "" H 2100 1550 50  0001 C CNN
+	1    2100 1550
+	1    0    0    -1
+$EndComp
+Wire Wire Line
+	2000 1550 2100 1550
+$Comp
+L power:GND #PWR?
+U 1 1 5CACEF75
+P 2350 1400
+F 0 "#PWR?" H 2350 1150 50  0001 C CNN
+F 1 "GND" H 2355 1227 50  0000 C CNN
+F 2 "" H 2350 1400 50  0001 C CNN
+F 3 "" H 2350 1400 50  0001 C CNN
+	1    2350 1400
+	1    0    0    -1
+$EndComp
+Wire Wire Line
+	2000 1400 2350 1400
 $EndSCHEMATC

Commit message: schematice mostly complete
Parts:
- removed U1: ATTINY-1616MNR, Package_DFN_QFN:QFN-20-1EP_3x3mm_P0.45mm_EP1.6x1.6mm, symbol solar_light-rescue:ATTINY-1616MNR-solar_light
- added C1, C4: 1u, symbol Device:C_Small
- added C2, C6: 4u7, symbol Device:C_Small
- added C5: 2u2, symbol Device:C_Small
- added L1: 2.2uh, symbol Device:L_Small
- added SW1: SW_SPST, symbol Switch:SW_SPST
- added TP1: SWC, symbol Connector:TestPoint
- added TP2: SWD, symbol Connector:TestPoint
- added U1: ATSAMD21E18A-MU, QFN50P500X500X100-33N, symbol ATSAMD21E18A-MU:ATSAMD21E18A-MU
- added U3: ISL9113, symbol solar_light:ISL9113
- added U4: MIC3490-3v3, symbol solar_light:MIC3490-3v3
- gave numbers to parts that had none: 7
Connections:
- net GND: now also D1.3 (VSS), D2.3 (VSS), C1.2, C2.2, C4.2, C5.2, C6.2, SW1.1 (A), U1.10 (GND), U1.28 (GND), U1.33 (EP), U3.1 (PGND), U3.6 (AGND), U4.2 (GND)
- net VCC: now also C2.1, C4.1, L1.1, U3.5 (EN), U3.7 (VBAT), U4.3 (EN), U4.4 (IN)
- net 5v: now reaches D1.1 (VDD), D2.1 (VDD)
- net 5v: now also C6.1, U3.2 (Vout)
- net light: now reaches D1.4 (DIN)
- net light: now also U1.17 (PA16)
- new net: SW1.2 (B), U1.26 (~RESET~)
- new net: C1.1, U1.29 (VDDCORE)
- new net: TP2.1, U1.31 (PA30)
- new net: TP1.1, U1.32 (PA31)
- new net: L1.2, U3.8 (SW)
- new net 3v3: C5.1, U1.30 (VDDIN), U1.9 (VDDANA), U4.5 (OUT)
- no-connect marks 0 -> 1
Other:
- moved on the sheet: D1, D2

Commit message: schematic done; pcb started
Parts:
- removed U3: ISL9113, symbol solar_light:ISL9113
- added J3: breakout header, Connector_PinHeader_1.00mm:PinHeader_1x08_P1.00mm_Horizontal, symbol Connector:Conn_01x08_Female
- added J4: USB_B_Mini, Connector_USB:USB_Micro-B_Amphenol_10103594-0001LF_Horizontal, symbol Connector:USB_B_Mini
- added R2, R3: R_Small, Resistor_SMD:R_0603_1608Metric, symbol Device:R_Small
- added SW2: BRIGHTNESS, Button_Switch_THT:SW_PUSH_6mm, symbol Switch:SW_SPST
- added SW3: COLOR, Button_Switch_THT:SW_PUSH_6mm, symbol Switch:SW_SPST
- added U3: ISL9111, Package_TO_SOT_SMD:SOT-23-6, symbol solar_light:ISL9111
- C1, C2, C3, C4, C5, C6: footprint (none) -> Capacitor_SMD:C_0603_1608Metric
- D3: footprint (none) -> Diode_SMD:D_SOD-123
- J1, J2: footprint (none) -> Connector_PinHeader_1.00mm:PinHeader_1x02_P1.00mm_Vertical
- L1: value 2.2uh -> 4.7uH; footprint (none) -> Resistor_SMD:R_0603_1608Metric_Pad1.05x0.95mm_HandSolder
- R1: footprint (none) -> Resistor_SMD:R_0603_1608Metric
- SW1: footprint (none) -> Button_Switch_THT:SW_PUSH_6mm
- TP1, TP2: footprint (none) -> TestPoint:TestPoint_Pad_D1.5mm
- U1: footprint QFN50P500X500X100-33N -> Package_DFN_QFN:QFN-32-1EP_5x5mm_P0.5mm_EP3.6x3.6mm
- U4: footprint (none) -> Package_TO_SOT_SMD:SOT-23-5
Connections:
- net 5v: now also C2.1, U3.5 (Vout); no longer C6.1
- net GND: now also J4.5 (GND), J4.6 (Shield), U3.2 (GND)
- net VCC: now also C6.1, L1.2, J4.1 (VBUS), U3.3 (EN), U3.6 (Vin); no longer C2.1, L1.1
- net at U1.1 (PA00): now also J3.1 (Pin_1)
- net at U1.18 (PA17): now also SW3.2 (B)
- net at U1.19 (PA18): now also SW3.1 (A)
- net at U1.2 (PA01): now also J3.2 (Pin_2)
- net at U1.20 (PA19): now also SW2.1 (A)
- net at U1.21 (PA22): now also SW2.2 (B)
- net D-: now reaches U1.23 (PA24)
- net D-: now also R3.2
- net D+: now reaches U1.24 (PA25)
- net D+: now also R2.1
- net at U1.3 (PA02): now also J3.3 (Pin_3)
- net at U1.4 (PA03): now also J3.4 (Pin_4)
- net at U1.5 (PA04): now also J3.5 (Pin_5)
- net at U1.6 (PA05): now also J3.6 (Pin_6)
- net at U1.7 (PA06): now also J3.7 (Pin_7)
- net at U1.8 (PA07): now also J3.8 (Pin_8)
- new net: L1.1, U3.1 (SW)
- new net: J4.2 (D-), R3.1
- new net: J4.3 (D+), R2.2
Other:
- moved on the sheet: L1

Commit message: routed!
Parts:
- J4: footprint Connector_USB:USB_Micro-B_Amphenol_10103594-0001LF_Horizontal -> Connector_USB:USB_Micro-B_Amphenol_10103594-0001LF_Horizontal-no-th
- SW1, SW2, SW3: footprint Button_Switch_THT:SW_PUSH_6mm -> Button_Switch_THT:SW_PUSH_3.5mm
Changed lines of the file:
@@
 F 0 "SW1" H 1000 1785 50  0000 C CNN
 F 1 "SW_SPST" H 1000 1694 50  0000 C CNN
-F 2 "Button_Switch_THT:SW_PUSH_6mm" H 1000 1550 50  0001 C CNN
+F 2 "Button_Switch_THT:SW_PUSH_3.5mm" H 1000 1550 50  0001 C CNN
 F 3 "" H 1000 1550 50  0001 C CNN
 	1    1000 1550
@@
 F 0 "SW2" H 4050 2835 50  0000 C CNN
 F 1 "BRIGHTNESS" H 4050 2744 50  0000 C CNN
-F 2 "Button_Switch_THT:SW_PUSH_6mm" H 4050 2600 50  0001 C CNN
+F 2 "Button_Switch_THT:SW_PUSH_3.5mm" H 4050 2600 50  0001 C CNN
 F 3 "" H 4050 2600 50  0001 C CNN
 	1    4050 2600
@@
 F 0 "SW3" H 4050 3185 50  0000 C CNN
 F 1 "COLOR" H 4050 3094 50  0000 C CNN
-F 2 "Button_Switch_THT:SW_PUSH_6mm" H 4050 2950 50  0001 C CNN
+F 2 "Button_Switch_THT:SW_PUSH_3.5mm" H 4050 2950 50  0001 C CNN
 F 3 "" H 4050 2950 50  0001 C CNN
 	1    4050 2950
@@
 F 0 "J4" H 7255 3817 50  0000 C CNN
 F 1 "USB_B_Mini" H 7255 3726 50  0000 C CNN
-F 2 "Connector_USB:USB_Micro-B_Amphenol_10103594-0001LF_Horizontal" H 7350 3300 50  0001 C CNN
+F 2 "Connector_USB:USB_Micro-B_Amphenol_10103594-0001LF_Horizontal-no-th" H 7350 3300 50  0001 C CNN
 F 3 "~" H 7350 3300 50  0001 C CNN
 	1    7200 3350
